Commit message: fix the franka_description

File: composite_robot_description/urdf/mobile_manipulator.urdf.xacro (robot description, xacro)
@@ -18,25 +18,7 @@
     <xacro:wheel_assembly_b prefix="rear_left_wheel" parent_link="base_link" x="-0.23" y="0.206" z="-0.1" roll="0" pitch="0" yaw="3.14159"/>
     <xacro:wheel_assembly_a prefix="rear_right_wheel" parent_link="base_link" x="-0.23" y="-0.206" z="-0.1" roll="0" pitch="0" yaw="3.14159"/>
-    <xacro:franka_arm parent_link="base_link" xyz="0.0 0 0.00" rpy="0 0 0"/>
-    <xacro:franka_hand connected_to="fr3_link8" safety_distance="0.03" arm_id="fr3" ee_id="franka_hand_white" ee_inertials="${hand_inertials}"/>
+    <xacro:franka_arm parent_link="base_link" xyz="0.0 0 0.00" rpy="0 0 0" />
+    <xacro:franka_hand connected_to="fr3_link8" safety_distance="0.03"  ee_id="franka_hand_white" ee_inertials="${hand_inertials}" robot_type="fr3"/>
     <ros2_control name="FrankaHandFakeSystem" type="system">
-        <hardware>
-            <plugin>gazebo_ros2_control/GazeboSystem</plugin>
-        </hardware>
-        <joint name="fr3_finger_joint1">
-            <command_interface name="position"/>
-            <state_interface name="position">
-              <param name="initial_value">0.0</param>
-            </state_interface>
-            <state_interface name="velocity"/>
-        </joint>
-        <joint name="fr3_finger_joint2">
-            <command_interface name="position"/>
-            <state_interface name="position">
-              <param name="initial_value">0.0</param>
-            </state_interface>
-            <state_interface name="velocity"/>
-        </joint>
-    </ros2_control><ros2_control name="FrankaHandFakeSystem" type="system">
         <hardware>
             <plugin>gazebo_ros2_control/GazeboSystem</plugin>
